File: KiCADWork/Dock/Charging.kicad_sch (KiCad schematic)
At the start: 9 parts, among them U1 MCP73831T-2ACI/OT, U2 XB6096I2SV

Commit message: New Chip NRF52833
large changes
Parts:
- removed C1, C3: 10u, Capacitor_SMD:C_0402_1005Metric_Pad0.74x0.62mm_HandSolder, symbol Device:C
- removed C2: 100n, Capacitor_SMD:C_0402_1005Metric_Pad0.74x0.62mm_HandSolder, symbol Device:C
- removed D1: WHITE LED, LED_SMD:LED_0603_1608Metric_Pad1.05x0.95mm_HandSolder, symbol Device:LED
- removed R1, R3: 2k, Resistor_SMD:R_0402_1005Metric_Pad0.72x0.64mm_HandSolder, symbol Device:R
- removed R2: 100, Resistor_SMD:R_0402_1005Metric_Pad0.72x0.64mm_HandSolder, symbol Device:R
- removed U1: MCP73831T-2ACI/OT, easyeda2kicad:SOT-23-5_L3.0-W1.7-P0.95-LS2.8-BL, symbol easyeda2kicad:MCP73831T-2ACI_OT
- removed U2: XB6096I2SV, easyeda2kicad:WDFN-6_L2.0-W2.0-P0.65-BL-EP, symbol easyeda2kicad:XB6096I2SV
