File: KiCADWork/Dock/DeviceSelect.kicad_sch (KiCad schematic)
At the start: 14 parts, among them SW1 SW_DIP_x01, SW2 SW_DIP_x01, U1 USB2422T-I/MJ, Y1 Crystal_GND24

Commit message: Dock Updates
Parts:
- removed C5, C6: 100n, Capacitor_SMD:C_0402_1005Metric_Pad0.74x0.62mm_HandSolder, symbol Device:C
- removed D3: WHITE LED, LED_SMD:LED_0603_1608Metric_Pad1.05x0.95mm_HandSolder, symbol Device:LED
- removed SW1, SW2: SW_DIP_x01, easyeda2kicad:KEY-SMD_L3.0-W2.5-LS4.0, symbol Switch:SW_DIP_x01
- added C10, C3, C7, C9: 100n, Capacitor_SMD:C_0402_1005Metric_Pad0.74x0.62mm_HandSolder, symbol Device:C
- added C11, C4, C8: 1u, Capacitor_SMD:C_0402_1005Metric_Pad0.74x0.62mm_HandSolder, symbol Device:C
- added D1: LED, LED_SMD:LED_0603_1608Metric_Pad1.05x0.95mm_HandSolder, symbol Device:LED
- added Q1: NTJD4152PT1G, easyeda2kicad:SC-88-6_L2.0-W1.3-P0.65-LS2.1-BL, symbol easyeda2kicad:NTJD4152PT1G
- added R10, R11: 2k, Resistor_SMD:R_0402_1005Metric_Pad0.72x0.64mm_HandSolder, symbol Device:R
- added R3: 10k, Resistor_SMD:R_0402_1005Metric_Pad0.72x0.64mm_HandSolder, symbol Device:R
- added R6, R7, R8: 100, Resistor_SMD:R_0402_1005Metric_Pad0.72x0.64mm_HandSolder, symbol Device:R
- added R9: 12k 1%, Resistor_SMD:R_0402_1005Metric_Pad0.72x0.64mm_HandSolder, symbol Device:R
- C1, C2: value 8p -> 18p
- D2: value BLUE LED -> LED
- R12, R13: value 2k -> 220
- Y1: value Crystal_GND24 -> X322524MOB4SI; footprint easyeda2kicad:CRYSTAL-SMD_4P-L2.0-W1.6-BL -> easyeda2kicad:CRYSTAL-SMD_4P-L3.2-W2.5-BL
Connections:
- net BLE2Sel is gone; now on net GND: D2.1 (K)
- net +3V3: now also C3.2, C4.2, C7.2, R3.2; no longer R12.2, R13.2
- net GND: now also C10.1, C11.1, C3.1, C4.1, C7.1, C8.1, C9.1, D1.1 (K), R6.1, R7.1, R8.1, R9.1
- net VBus: now also Q1.1 (S1), Q1.4 (S2), R10.1, R11.1
- net at U1.10 (CRFILT): now also C8.2
- net PWREN2: now reaches U1.11 (PRTPWR2)
- net PWREN2: now also Q1.5 (G2), R11.2
- net at U1.13 (SMBDATA/NON_REM1): now also R6.2
- net at U1.14 (SMBCLK/CFG_SEL0): now also R8.2
- net RESET: now reaches U1.15 (RESET_N)
- net RESET: now also C11.2, R3.1
- net at R1.1, R2.2, U1.16 (VBUS_DET): now also C10.2
- net at U1.17 (SUSP_IND/LOCAL_PWR/(NON_REM0)): now also R7.2
- net at U1.23 (PLLFILT): now also C9.2
- net at U1.24 (RBIAS): now also R9.2
- net PWREN1: now reaches U1.7 (PRTPWR1/(BC_EN1))
- net PWREN1: now also Q1.2 (G1), R10.2
- net VBUS1: now reaches R12.1
- net VBUS1: now also Q1.6 (D1)
- net at D2.2 (A): now also R13.2; no longer R13.1
- new net: D1.2 (A), R12.2
- new net VBUS2: Q1.3 (D2), R13.1
- no-connect marks 1 -> 3
Other:
- moved on the sheet: C1, C2, R1, R2, Y1

Commit message: Ignoring Backups
More Dock progress
All local backups removed
Parts:
- C1, C2: LCSC Part (none) -> C5137554
- C11, C4, C8: LCSC Part (none) -> C14445
- C3, C7, C9: LCSC Part (none) -> C60474
- D1, D2: value LED -> BLUE LED; LCSC Part (none) -> C7371904
- R1, R2: value 100 -> 10k
- R10, R11: LCSC Part (none) -> C60488
- R12, R13: LCSC Part (none) -> C112291
- R3: LCSC Part (none) -> C60490
- R6, R7, R8: LCSC Part (none) -> C3015757
- R9: value 12k 1% -> 12k; LCSC Part (none) -> C137923
- Y1: LCSC Part (none) -> C70590
Connections:
- net VBus: no longer R1.2
- new net Vsys: R1.2
Changed lines of the file:
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@@
     (stroke (width 0) (type default))
   )
-  (wire (pts (xy 79.375 123.825) (xy 67.945 123.825))
+  (wire (pts (xy 71.12 123.825) (xy 67.945 123.825))
     (stroke (width 0) (type default))
   )
@@
   (label "Earring2" (at 70.485 59.055 180) (fields_autoplaced)
     (effects (font (size 1.27 1.27)) (justify right bottom))
+  )
+  (label "USB HUB" (at 118.11 29.845 0) (fields_autoplaced)
+    (effects (font (size 3 3)) (justify left bottom))
   )
   (label "Cs=3p" (at 262.89 63.5 0) (fields_autoplaced)
@@
     (effects (font (size 1.27 1.27)) (justify left bottom))
   )
-  (label "Earring 2 charging" (at 107.95 153.035 270) (fields_autoplaced)
+  (label "MOSFET switch USB Power Path" (at 54.61 116.84 0) (fields_autoplaced)
+    (effects (font (size 3 3)) (justify left bottom))
+  )
+  (label "Earring 2 charging" (at 114.3 153.67 270) (fields_autoplaced)
     (effects (font (size 1.27 1.27)) (justify right bottom))
   )
@@
     (effects (font (size 1.27 1.27)) (justify left bottom))
   )
-  (global_label "PWREN2" (shape input) (at 85.09 74.295 180) (fields_autoplaced)
+  (global_label "PWREN2" (shape output) (at 85.09 74.295 180) (fields_autoplaced)
     (effects (font (size 1.27 1.27)) (justify right))
     (property "Intersheetrefs" "${INTERSHEET_REFS}" (at 74.4244 74.295 0)
@@
     )
   )
-  (global_label "PWREN1" (shape input) (at 85.09 64.135 180) (fields_autoplaced)
+  (global_label "PWREN1" (shape output) (at 85.09 64.135 180) (fields_autoplaced)
     (effects (font (size 1.27 1.27)) (justify right))
     (property "Intersheetrefs" "${INTERSHEET_REFS}" (at 74.4244 64.135 0)
@@
     (effects (font (size 1.27 1.27)) (justify left))
   )
-  (hierarchical_label "VBus" (shape bidirectional) (at 220.98 71.755 90) (fields_autoplaced)
+  (hierarchical_label "Vsys" (shape bidirectional) (at 220.98 71.755 90) (fields_autoplaced)
     (effects (font (size 1.27 1.27)) (justify left))
   )
-  (hierarchical_label "VBUS1" (shape bidirectional) (at 79.375 123.825 0) (fields_autoplaced)
+  (hierarchical_label "VBUS1" (shape bidirectional) (at 71.12 123.825 0) (fields_autoplaced)
     (effects (font (size 1.27 1.27)) (justify left))
   )
@@
     )
     (property "Datasheet" "~" (at 212.09 67.945 0)
+      (effects (font (size 1.27 1.27)) hide)
+    )
+    (property "LCSC Part" "C60474 " (at 212.09 67.945 0)
       (effects (font (size 1.27 1.27)) hide)
     )
@@
       (effects (font (size 1.27 1.27)) (justify right))
     )
-    (property "Value" "LED" (at 101.6 164.1475 90)
+    (property "Value" "BLUE LED" (at 101.6 164.1475 90)
       (effects (font (size 1.27 1.27)) (justify right))
     )
@@
       (effects (font (size 1.27 1.27)) hide)
     )
+    (property "LCSC Part" "C7371904 " (at 97.79 161.29 0)
+      (effects (font (size 1.27 1.27)) hide)
+    )
     (pin "2")
     (pin "1")
@@
       (effects (font (size 1.27 1.27)) hide)
     )
+    (property "LCSC Part" "C60474 " (at 54.61 41.275 0)
+      (effects (font (size 1.27 1.27)) hide)
+    )
     (pin "1")
     (pin "2")
@@
     )
     (property "Datasheet" "~" (at 48.895 127.635 0)
+      (effects (font (size 1.27 1.27)) hide)
+    )
+    (property "LCSC Part" "C112291" (at 48.895 127.635 0)
       (effects (font (size 1.27 1.27)) hide)
     )
@@
     )
     (property "Datasheet" "~" (at 247.65 100.965 0)
+      (effects (font (size 1.27 1.27)) hide)
+    )
+    (property "LCSC Part" "C60490 " (at 247.65 100.965 0)
       (effects (font (size 1.27 1.27)) hide)
     )
@@
       (effects (font (size 1.27 1.27)))
     )
-    (property "Value" "12k 1%" (at 198.755 46.355 90)
+    (property "Value" "12k" (at 198.755 46.355 90)
       (effects (font (size 1.27 1.27)))
     )
@@
     )
     (property "Datasheet" "~" (at 198.755 48.895 0)
+      (effects (font (size 1.27 1.27)) hide)
+    )
+    (property "LCSC Part" "C137923" (at 198.755 48.895 0)
       (effects (font (size 1.27 1.27)) hide)
     )
@@
       (effects (font (size 1.27 1.27)))
     )
-    (property "Value" "100" (at 218.44 89.535 90)
+    (property "Value" "10k" (at 218.44 89.535 90)
       (effects (font (size 1.27 1.27)))
     )
@@
     )
     (property "Datasheet" "~" (at 220.98 89.535 0)
+      (effects (font (size 1.27 1.27)) hide)
+    )
+    (property "LCSC Part" "" (at 220.98 89.535 0)
       (effects (font (size 1.27 1.27)) hide)
     )
@@
       (effects (font (size 1.27 1.27)) hide)
     )
+    (property "LCSC Part" "C70590 " (at 252.095 57.785 0)
+      (effects (font (size 1.27 1.27)) hide)
+    )
     (pin "1")
     (pin "2")
@@
       (effects (font (size 1.27 1.27)) hide)
     )
+    (property "LCSC Part" "C14445 " (at 71.12 76.2 0)
+      (effects (font (size 1.27 1.27)) hide)
+    )
     (pin "1")
     (pin "2")
@@
       (effects (font (size 1.27 1.27)) hide)
     )
+    (property "LCSC Part" "C14445 " (at 55.88 73.025 0)
+      (effects (font (size 1.27 1.27)) hide)
+    )
     (pin "1")
     (pin "2")
@@
     )
     (property "Datasheet" "~" (at 108.585 132.715 0)
+      (effects (font (size 1.27 1.27)) hide)
+    )
+    (property "LCSC Part" "C60488 " (at 108.585 132.715 0)
       (effects (font (size 1.27 1.27)) hide)
     )
@@
       (effects (font (size 1.27 1.27)) hide)
     )
+    (property "LCSC Part" "" (at 202.565 90.17 0)
+      (effects (font (size 1.27 1.27)) hide)
+    )
     (pin "1")
     (pin "2")
@@
     )
     (property "Datasheet" "~" (at 247.65 117.475 0)
+      (effects (font (size 1.27 1.27)) hide)
+    )
+    (property "LCSC Part" "C14445 " (at 247.65 117.475 0)
       (effects (font (size 1.27 1.27)) hide)
     )
@@
       (effects (font (size 1.27 1.27)) hide)
     )
+    (property "LCSC Part" "C3015757 " (at 179.07 93.98 0)
+      (effects (font (size 1.27 1.27)) hide)
+    )
     (pin "1")
     (pin "2")
@@
       (effects (font (size 1.27 1.27)) hide)
     )
+    (property "LCSC Part" "C3015757 " (at 183.515 83.82 0)
+      (effects (font (size 1.27 1.27)) hide)
+    )
     (pin "1")
     (pin "2")
@@
     )
     (property "Datasheet" "~" (at 212.725 43.18 0)
+      (effects (font (size 1.27 1.27)) hide)
+    )
+    (property "LCSC Part" "C60474 " (at 212.725 43.18 0)
       (effects (font (size 1.27 1.27)) hide)
     )
@@
       (effects (font (size 1.27 1.27)) hide)
     )
+    (property "LCSC Part" "C112291" (at 97.79 154.305 0)
+      (effects (font (size 1.27 1.27)) hide)
+    )
     (pin "1")
     (pin "2")
@@
       (effects (font (size 1.27 1.27)) hide)
     )
+    (property "LCSC Part" "C3015757 " (at 192.405 93.345 0)
+      (effects (font (size 1.27 1.27)) hide)
+    )
     (pin "1")
     (pin "2")
@@
       (effects (font (size 1.27 1.27)))
     )
-    (property "Value" "100" (at 218.44 77.47 90)
+    (property "Value" "10k" (at 218.44 77.47 90)
       (effects (font (size 1.27 1.27)))
     )
@@
     )
     (property "Datasheet" "~" (at 220.98 77.47 0)
+      (effects (font (size 1.27 1.27)) hide)
+    )
+    (property "LCSC Part" "" (at 220.98 77.47 0)
       (effects (font (size 1.27 1.27)) hide)
     )
@@
       (effects (font (size 1.27 1.27)) hide)
     )
+    (property "LCSC Part" "C5137554" (at 243.84 69.215 0)
+      (effects (font (size 1.27 1.27)) hide)
+    )
     (pin "1")
     (pin "2")
@@
     )
     (property "Datasheet" "~" (at 74.295 146.685 0)
+      (effects (font (size 1.27 1.27)) hide)
+    )
+    (property "LCSC Part" "C60488 " (at 74.295 146.685 0)
       (effects (font (size 1.27 1.27)) hide)
     )
@@
     )
     (property "Datasheet" "~" (at 244.475 53.975 0)
+      (effects (font (size 1.27 1.27)) hide)
+    )
+    (property "LCSC Part" "C5137554" (at 244.475 53.975 0)
       (effects (font (size 1.27 1.27)) hide)
     )
@@
       (effects (font (size 1.27 1.27)) (justify right))
     )
-    (property "Value" "LED" (at 52.705 137.4775 90)
+    (property "Value" "BLUE LED" (at 52.705 137.4775 90)
       (effects (font (size 1.27 1.27)) (justify right))
     )
@@
       (effects (font (size 1.27 1.27)) hide)
     )
+    (property "LCSC Part" "C7371904 " (at 48.895 134.62 0)
+      (effects (font (size 1.27 1.27)) hide)
+    )

Commit message: Beautiful Skilkscreen Added
Dock schematic intial draft complete
Parts:
- added TP1 (x3): TestPoint, TestPoint:TestPoint_Pad_D1.0mm, symbol Connector:TestPoint
Connections:
- net PWREN1: now also TP1.1
- net PWREN2: now also TP1.1
- net VBus: now also TP1.1
Other:
- moved on the sheet: C8, D1, R12

Commit message: Initial Dock DRC Complete
Parts:
- removed Q1: NTJD4152PT1G, easyeda2kicad:SC-88-6_L2.0-W1.3-P0.65-LS2.1-BL, symbol easyeda2kicad:NTJD4152PT1G
- removed R10, R11: 2k, Resistor_SMD:R_0402_1005Metric_Pad0.72x0.64mm_HandSolder, symbol Device:R
- removed TP1 (x3): TestPoint, TestPoint:TestPoint_Pad_D1.0mm, symbol Connector:TestPoint
- added C20, C22: 100n, Capacitor_SMD:C_0402_1005Metric_Pad0.74x0.62mm_HandSolder, symbol Device:C
- added C21, C23: 4.7u, Capacitor_SMD:C_0402_1005Metric_Pad0.74x0.62mm_HandSolder, symbol Device:C
- added TP1 (x2): TestPoint, TestPoint:TestPoint_Pad_D1.0mm, symbol Connector:TestPoint
- added U5, U6: SIP32509DT-T1-GE3, Package_TO_SOT_SMD:SOT-23-6_Handsoldering, symbol easyeda2kicad:SIP32509DT-T1-GE3
- U1: footprint Temp:QFN-24_L4.0-W4.0-P0.50-TL-EP2.5 -> Package_DFN_QFN:HVQFN-24-1EP_4x4mm_P0.5mm_EP2.5x2.5mm_ThermalVias
Connections:
- net D1+: now also U1.5 (USBDP_DN2/PRT_DIS_P2); no longer U1.3 (USBDP_DN1/PRT_DIS_P1)
- net D1-: now also U1.4 (USBDM_DN2/PRT_DIS_M2); no longer U1.2 (USBDM_DN1/PRT_DIS_M1)
- net D2+: now also U1.3 (USBDP_DN1/PRT_DIS_P1); no longer U1.5 (USBDP_DN2/PRT_DIS_P2)
- net D2-: now also U1.2 (USBDM_DN1/PRT_DIS_M1); no longer U1.4 (USBDM_DN2/PRT_DIS_M2)
- net GND: now also U1.25 (EP), C21.1, C23.1, U5.4 (GND), U6.4 (GND)
- net PWREN1: now also U1.11 (PRTPWR2), C20.1, U5.3 (EN); no longer U1.7 (PRTPWR1/(BC_EN1))
- net PWREN2: now also U1.7 (PRTPWR1/(BC_EN1)), C22.1, U6.3 (EN); no longer U1.11 (PRTPWR2)
- net VBUS1: now also C20.2, TP1.1, U5.1 (OUT), U5.2 (OUT)
- net VBUS2: now also C22.2, TP1.1, U6.1 (OUT), U6.2 (OUT)
- net Vsys: now also C21.2, C23.2, U5.5 (IN), U5.6 (IN), U6.5 (IN), U6.6 (IN)
Other:
- moved on the sheet: D1, R12
