File: KiCADWork/Dock/Dock.kicad_pcb (KiCad board)
At the start: 2 copper layers, 42.3 x 54.4 mm, 70 parts, among them J1 USB_C_Receptacle, J4 Conn_01x10_Socket, P1 USB_C_Plug, P2 USB_C_Plug, Q1 NTJD4152PT1G, U1 USB2422T-I/MJ, U2 TPS61023DRLR, U3 AMS1117-3.3, U4 BQ24073RGT, Y1 X322524MOB4SI

Commit message: Initial Dock DRC Complete
Parts:
- removed Q1: NTJD4152PT1G, easyeda2kicad:SC-88-6_L2.0-W1.3-P0.65-LS2.1-BL
- removed TP1, TP2, TP5: TestPoint, TestPoint:TestPoint_Pad_D1.0mm
- added C18: 100n, Capacitor_SMD:C_0402_1005Metric_Pad0.74x0.62mm_HandSolder, F.Cu at (122.4, 66.6)
- added C19: 100n, Capacitor_SMD:C_0402_1005Metric_Pad0.74x0.62mm_HandSolder, F.Cu at (168.7, 59.8)
- added C20: 100n, Capacitor_SMD:C_0402_1005Metric_Pad0.74x0.62mm_HandSolder, F.Cu at (140.8, 66.4)
- added C21: 4.7u, Capacitor_SMD:C_0402_1005Metric_Pad0.74x0.62mm_HandSolder, F.Cu at (134.9, 66.4)
- added C22: 100n, Capacitor_SMD:C_0402_1005Metric_Pad0.74x0.62mm_HandSolder, F.Cu at (148.8, 70.8)
- added C23: 4.7u, Capacitor_SMD:C_0402_1005Metric_Pad0.74x0.62mm_HandSolder, F.Cu at (148.3, 76.7)
- added G***: LOGO, easyeda2kicad:OTS2, F.Cu at (144.5, 95.8)
- added R22: 1k, Resistor_SMD:R_0402_1005Metric_Pad0.72x0.64mm_HandSolder, B.Cu at (122.4, 66.6)
- added R23: 1k, Resistor_SMD:R_0402_1005Metric_Pad0.72x0.64mm_HandSolder, B.Cu at (168.7, 59.8)
- added U5: SIP32509DT-T1-GE3, Package_TO_SOT_SMD:SOT-23-6_Handsoldering, F.Cu at (137.9, 66.9)
- added U6: SIP32509DT-T1-GE3, Package_TO_SOT_SMD:SOT-23-6_Handsoldering, F.Cu at (148.8, 73.7)
- BT2: footprint easyeda2kicad:CONN-TH_S2B-PH-K-LF-SN -> easyeda2kicad:CONN-TH_S2B-PH-K-S-LF-SN
- R10, R11: value 2k -> 0R; footprint Resistor_SMD:R_0402_1005Metric_Pad0.72x0.64mm_HandSolder -> Resistor_SMD:R_0805_2012Metric_Pad1.20x1.40mm_HandSolder
- R5: moved to B.Cu
- U1: footprint Temp:QFN-24_L4.0-W4.0-P0.50-TL-EP2.5 -> Package_DFN_QFN:HVQFN-24-1EP_4x4mm_P0.5mm_EP2.5x2.5mm_ThermalVias
- moved TP3 114.5 mm to (127.2, 65.4)
- moved D2 95.3 mm to (148.6, 68.3), turned to 180 degrees
- moved R13 91.1 mm to (148.8, 69.8), turned to 180 degrees
- moved D1 89.8 mm to (143.1, 66.9), turned to 180 degrees
- moved TP4 86.0 mm to (159.0, 69.8)
- moved R12 84.2 mm to (141.6, 68.2)
- moved R10 79.8 mm to (146.6, 89.6), turned to 180 degrees
- moved R11 78.9 mm to (145.6, 91.5), turned to 180 degrees
- moved TP17 68.3 mm to (154.0, 94.7), turned to 90 degrees
- moved TP11 67.6 mm to (151.6, 93.5), turned to 90 degrees
- moved D4 61.0 mm to (133.9, 101.2), turned to 160 degrees
- moved R14 56.8 mm to (129.6, 93.0), turned to -90 degrees
- moved R18 56.7 mm to (130.8, 94.2), turned to 90 degrees
- moved TP8 56.0 mm to (132.4, 95.2), turned to 180 degrees
- moved P1 54.7 mm to (120.3, 63.1), turned to -90 degrees
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Connections:
- J1 pad A6: /DeviceSelect/D+ -> Net-(J1-D+-PadA6)
- J1 pad A7: /DeviceSelect/D+ -> Net-(J1-D--PadA7)
- J1 pad B10: /DeviceSelect/D+ -> unconnected-(J1-RX1--PadB10)
- J1 pad B11: /DeviceSelect/D+ -> unconnected-(J1-RX1+-PadB11)
- J1 pad B6: /DeviceSelect/D+ -> Net-(J1-D+-PadA6)
- J1 pad B7: /DeviceSelect/D+ -> Net-(J1-D--PadA7)
- P1 pad S1: GND -> Net-(P1-SHIELD)
- P2 pad S1: GND -> Net-(P2-SHIELD)
- R10 pad 1: /DeviceSelect/VBus -> /DeviceSelect/D+
- R10 pad 2: PWREN1 -> Net-(J1-D+-PadA6)
- R11 pad 1: /DeviceSelect/VBus -> Net-(J1-D--PadA7)
- R11 pad 2: PWREN2 -> /DeviceSelect/D-
- TP3 pad 1: PWREN2 -> /DeviceSelect/VBUS1
- TP4 pad 1: PWREN1 -> /DeviceSelect/VBUS2
- U1 pad 11: PWREN2 -> PWREN1
- U1 pad 19: /DeviceSelect/D+ -> /DeviceSelect/D-
- U1 pad 2: /DeviceSelect/D1- -> /DeviceSelect/D2-
- U1 pad 25: unconnected-(U1-EP-Pad25) -> GND
- U1 pad 3: /DeviceSelect/D1+ -> /DeviceSelect/D2+
- U1 pad 4: /DeviceSelect/D2- -> /DeviceSelect/D1-
- U1 pad 5: /DeviceSelect/D2+ -> /DeviceSelect/D1+
- U1 pad 7: PWREN1 -> PWREN2
Routing:
- net GND: track 34.9 -> 102.7 mm, vias 32 -> 60
- net SWDIO: track 70.0 -> 132.3 mm
- net nRESET: track 57.5 -> 112.8 mm, vias 2 -> 3
- net SWO: track 66.1 -> 117.6 mm, vias 2 -> 3
- net SWCLK: track 71.2 -> 117.4 mm, vias 2 -> 3
- net /DeviceSelect/D1-: track 5.34 -> 45.4 mm
- net /DeviceSelect/D1+: track 5.09 -> 45.0 mm
- net +3V3: track 6.86 -> 43.4 mm, vias 0 -> 5
- net VTRef: track 16.8 -> 51.8 mm
- net /DeviceSelect/Vsys: track 14.5 -> 46.2 mm, vias 0 -> 3
- net PWREN1: track 0.00 -> 26.3 mm, vias 0 -> 2
- net /DeviceSelect/VBUS2: track 12.2 -> 38.2 mm, vias 2 -> 4
- net /DeviceSelect/D2+: track 5.09 -> 28.7 mm
- net /DeviceSelect/D2-: track 5.34 -> 28.5 mm
- net /DeviceSelect/VBUS1: track 12.1 -> 35.1 mm
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- added copper zone on F.Cu, net VTRef
Other:
- board size 42.3 x 54.4 mm -> 54.4 x 42.8 mm
- board text added: "DKD"
- board text added: "V1"
- board text added: "VBUS1"
