File: KiCADWork/Dock/Dock.kicad_pcb (KiCad board)
At the start: 2 copper layers, 54.4 x 42.8 mm, 77 parts, among them J1 USB_C_Receptacle, J4 Conn_01x10_Socket, P1 USB_C_Plug, P2 USB_C_Plug, U1 USB2422T-I/MJ, U2 TPS61023DRLR, U3 AMS1117-3.3, U4 BQ24073RGT, U5 SIP32509DT-T1-GE3, U6 SIP32509DT-T1-GE3, Y1 X322524MOB4SI

Commit message: Started mirror earrings and case
Other:
- board text added: "locked"
- board text removed: "DKD"
- board text removed: "V1"
- board text removed: "VBUS1"
