File: KiCADWork/BLEEarrings nRF52832/BLEEarrings.kicad_pcb (KiCad board)
At the start: 2 copper layers, 25.5 x 37.8 mm, 48 parts, among them J1 Screw_Terminal_01x01, J2 Screw_Terminal_01x02, J3 USB_C_Receptacle, SW1 TK-6580B-1, SW2 SW_DIP_x01, U1 MCP73831T-2ACI/OT, U2 XB6096I2SV, U3 NRF52833-QDAA-R7, Y1 XL7EL89CKI-111YLC-32M, Y2 X161032768KLD2SI

Commit message: Ignoring Backups
More Dock progress
All local backups removed
Parts:
- added G***: LOGO, CustomPads:DK6, B.Cu at (145.8, 58.4)
- added R5: NF, Resistor_SMD:R_0201_0603Metric, F.Cu at (142.8, 60.2)
- added R6: NF, Resistor_SMD:R_0201_0603Metric, F.Cu at (143.5, 60.6)
- added R7: NF, Resistor_SMD:R_0201_0603Metric, F.Cu at (148.1, 60.5)
- added R8: NF, Resistor_SMD:R_0201_0603Metric, F.Cu at (146.9, 60.7)
- added TP1: TestPoint, TestPoint:TestPoint_Pad_D1.0mm, F.Cu at (147.4, 46.4)
- moved TP16 14.2 mm to (135.2, 49.8)
- moved TP9 10.6 mm to (145.6, 45.4)
- moved R13 8.03 mm to (144.6, 48.0), turned to 0 degrees
- moved C18 6.37 mm to (141.1, 44.0), turned to 0 degrees
- moved C13 6.03 mm to (130.6, 44.9), turned to 90 degrees
- moved R14 5.40 mm to (144.6, 49.0)
- moved R4 4.89 mm to (136.4, 44.3), turned to -90 degrees
- moved R3 4.51 mm to (141.1, 42.9)
- moved C4 4.43 mm to (147.4, 48.4)
- moved U2 4.28 mm to (141.1, 45.9), turned to -90 degrees
- moved R2 3.71 mm to (144.0, 46.1), turned to 90 degrees
- moved C3 3.50 mm to (147.4, 52.8)
- moved C19 3.46 mm to (135.4, 45.4), turned to 90 degrees
- moved TP10 2.11 mm to (141.1, 70.9)
- moved D2 1.62 mm to (139.8, 66.2)
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Connections:
- J3 pad A10: nRESET -> /DSP/nReset
- J3 pad A11: SWO -> SWO_L
- J3 pad A2: SWDIO -> SWDIO_L
- J3 pad A3: SWDCLK -> SWDCLK_L
- J3 pad B10: nRESET -> /DSP/nReset
- J3 pad B11: SWO -> SWO_L
- J3 pad B2: SWDIO -> SWDIO_L
- J3 pad B3: SWDCLK -> SWDCLK_L
- U3 pad 16: nRESET -> Net-(U3-P0.18_nRESET)
- U3 pad 17: SWO -> Net-(U3-P0.20)
- U3 pad 19: SWDCLK -> Net-(U3-SWDIO)
- U3 pad 20: SWDIO -> Net-(U3-SWDCLK)
- U3 pad 33: BatRef -> NEO_LED
- U3 pad 34: NEO_LED -> BatRef
Routing:
- net +3V3: track 1.88 -> 54.1 mm, vias 0 -> 6
- net GND: track 12.9 -> 48.4 mm, vias 8 -> 29
- net /DSP/VBUS: track 27.0 -> 59.1 mm, vias 4 -> 6
- net nRESET: track 22.5 -> 0.00 mm, vias 2 -> 0
- net SWDIO_L: track 0.00 -> 22.1 mm, vias 0 -> 3
- net SWO: track 22.0 -> 0.00 mm, vias 2 -> 0
- net SWDIO: track 21.1 -> 0.00 mm, vias 2 -> 0
- net SWDCLK: track 19.0 -> 0.00 mm, vias 3 -> 0
- net /DSP/nReset: track 0.00 -> 18.7 mm, vias 0 -> 2
- net SWDCLK_L: track 0.00 -> 16.9 mm, vias 0 -> 2
- net SWO_L: track 0.00 -> 16.9 mm, vias 0 -> 3
- net DEC6: track 2.18 -> 16.2 mm, vias 0 -> 2
- net +BATT: track 13.9 -> 23.8 mm, vias 1 -> 2
- net /Power/VBAT: track 22.2 -> 14.9 mm
- net Net-(U1-STAT): track 2.66 -> 7.54 mm
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Other:
- board size 25.5 x 37.8 mm -> 25.8 x 38.8 mm
- board text added: "+"
- board text added: "-"
- board text added: "0V"
- board text added: "3V3"
- board text added: "Bat+"
- board text added: "BatRef"
- board text added: "DK"
- board text added: "LED"
- board text added: "RST"
- board text added: "SWDIO"
- board text added: "SWO"
- board text added: "V1"
- board text added: "o o ← Brainwashing Rays → o"

Commit message: Beautiful Skilkscreen Added
Dock schematic intial draft complete
Parts:
- removed the G*** at (145.8, 58.4)
- removed TP1: TestPoint, TestPoint:TestPoint_Pad_D1.0mm
- added G***: LOGO, CustomPads:OT2, B.Cu at (144.3, 59.1)
- added R10: 5k1, Resistor_SMD:R_0402_1005Metric_Pad0.72x0.64mm_HandSolder, F.Cu at (140.3, 68.6)
- added R11: 5k1, Resistor_SMD:R_0402_1005Metric_Pad0.72x0.64mm_HandSolder, F.Cu at (148.8, 64.1)
- D1: value WHITE LED -> RED LED
Connections:
- J3 pad A5: GND -> Net-(J3-CC1)
- J3 pad B5: GND -> Net-(J3-CC2)
Routing:
- net GND: track 48.4 -> 38.4 mm
- net Net-(J3-CC2): track 0.00 -> 5.09 mm
- net Net-(J3-CC1): track 0.00 -> 3.14 mm

Commit message: Initial Dock DRC Complete
Parts:
- BT1: footprint easyeda2kicad:CONN-TH_1.25-2AW -> easyeda2kicad:CONN-TH_530480210
Routing:
- net GND: vias 29 -> 33
Changed lines of the file:
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@@
     (descr "Resistor SMD 0402 (1005 Metric), square (rectangular) end terminal, IPC_7351 nominal with elongated pad for handsoldering. (Body size source: IPC-SM-782 page 72, https://www.pcb-3d.com/wordpress/wp-content/uploads/ipc-sm-782a_amendment_1_and_2.pdf), generated with kicad-footprint-generator")
     (tags "resistor handsolder")
-    (property "LCSC Part" "C105872")
+    (property "LCSC Part" "C103086")
     (property "Sheetfile" "BLEEarrings.kicad_sch")
     (property "Sheetname" "")
@@
     (descr "Resistor SMD 0402 (1005 Metric), square (rectangular) end terminal, IPC_7351 nominal with elongated pad for handsoldering. (Body size source: IPC-SM-782 page 72, https://www.pcb-3d.com/wordpress/wp-content/uploads/ipc-sm-782a_amendment_1_and_2.pdf), generated with kicad-footprint-generator")
     (tags "resistor handsolder")
-    (property "LCSC Part" "C105872")
+    (property "LCSC Part" "C103086")
     (property "Sheetfile" "BLEEarrings.kicad_sch")
     (property "Sheetname" "")
@@
     )
   )
-  (footprint "easyeda2kicad:CONN-TH_1.25-2AW" (layer "B.Cu")
+  (footprint "easyeda2kicad:CONN-TH_530480210" (layer "B.Cu")
     (at 144.18 43.28 180)
     (property "LCSC Part" "C173752")
@@
     (property "ki_keywords" "batt voltage-source cell")
     (attr through_hole)
-    (fp_text reference "BT1" (at -3.27 -1.54 270) (layer "B.SilkS")
+    (fp_text reference "BT1" (at 0 4) (layer "B.SilkS")
         (effects (font (size 1 1) (thickness 0.15)) (justify mirror))
     )
@@
         (effects (font (size 1 1) (thickness 0.15)) (justify mirror))
     )
-    (fp_line (start -2.2 -4) (end -2.2 0.8)
+    (fp_line (start -2.12 1.05) (end -2.12 -4.45)
       (stroke (width 0.25) (type solid)) (layer "B.SilkS"))
-    (fp_line (start -2.2 -4) (end 2.2 -4)
+    (fp_line (start -2.12 1.05) (end -1.25 1.05)
       (stroke (width 0.25) (type solid)) (layer "B.SilkS"))
-    (fp_line (start -2.2 0.8) (end -1.25 0.8)
+    (fp_line (start -1.25 1.05) (end -1.25 0.38)
       (stroke (width 0.25) (type solid)) (layer "B.SilkS"))
-    (fp_line (start -1.25 0.27) (end -1.25 0.27)
+    (fp_line (start 1.29 1.02) (end 1.29 0.34)
       (stroke (width 0.25) (type solid)) (layer "B.SilkS"))
-    (fp_line (start -1.25 0.8) (end -1.25 0.27)
+    (fp_line (start 2.16 -4.44) (end -2.12 -4.44)
       (stroke (width 0.25) (type solid)) (layer "B.SilkS"))
-    (fp_line (start 1.25 0.27) (end 1.25 0.27)
+    (fp_line (start 2.16 1.02) (end 1.29 1.02)
       (stroke (width 0.25) (type solid)) (layer "B.SilkS"))
-    (fp_line (start 1.25 0.8) (end 1.25 0.27)
+    (fp_line (start 2.16 1.02) (end 2.16 -4.44)
       (stroke (width 0.25) (type solid)) (layer "B.SilkS"))
-    (fp_line (start 2.2 -4) (end 2.2 0.8)
-      (stroke (width 0.25) (type solid)) (layer "B.SilkS"))
-    (fp_line (start 2.2 0.8) (end 1.25 0.8)
-      (stroke (width 0.25) (type solid)) (layer "B.SilkS"))
-    (fp_rect (start -6 -4) (end 6 -52.6)
-      (stroke (width 0.2) (type default)) (fill none) (layer "Cmts.User"))
-    (fp_circle (center -2.33 -4.13) (end -2.3 -4.13)
+    (fp_rect (start -5.98 -4.74) (end 6.02 -53.34)
+      (stroke (width 0.2) (type default)) (fill none) (layer "B.SilkS"))
+    (fp_circle (center -2.25 -4.58) (end -2.22 -4.58)
       (stroke (width 0.06) (type solid)) (fill none) (layer "B.Fab"))
-    (fp_circle (center -0.63 0) (end -0.55 0)
-      (stroke (width 0.15) (type solid)) (fill none) (layer "B.Fab"))
-    (fp_circle (center 0.63 0) (end 0.71 0)
-      (stroke (width 0.15) (type solid)) (fill none) (layer "B.Fab"))
-    (pad "1" thru_hole circle (at -0.62 0 180) (size 0.9 0.9) (drill 0.500024) (layers "*.Cu" "*.Mask")
+    (fp_circle (center -0.62 0) (end -0.52 0)
+      (stroke (width 0.2) (type solid)) (fill none) (layer "B.Fab"))
+    (fp_circle (center 0.62 0) (end 0.72 0)
+      (stroke (width 0.2) (type solid)) (fill none) (layer "B.Fab"))
+    (pad "1" thru_hole rect (at -0.62 0 180) (size 1 1) (drill 0.599999) (layers "*.Cu" "*.Mask")
       (net 23 "Net-(BT1-+)") (pinfunction "+") (pintype "passive"))
-    (pad "2" thru_hole circle (at 0.62 0 180) (size 0.9 0.9) (drill 0.500024) (layers "*.Cu" "*.Mask")
+    (pad "2" thru_hole circle (at 0.62 0 180) (size 1 1) (drill 0.599999) (layers "*.Cu" "*.Mask")
       (net 10 "Net-(BT1--)") (pinfunction "-") (pintype "passive"))
-    (model "C:/BLEEarrings/CADWork/Battery/BatteryGens.STEP"
-      (offset (xyz 0 -2.4 0))
+    (model "C:/BLEEarrings/CADWork/Battery/Earring/BatteryGens.STEP"
+      (offset (xyz 0 -3.3 0))
       (scale (xyz 1 1 1))
       (rotate (xyz -90 0 0))
@@
   (via (at 149.51 43.90125) (size 0.7) (drill 0.3) (layers "F.Cu" "B.Cu") (net 1))
   (via (at 149.51 53.08) (size 0.7) (drill 0.3) (layers "F.Cu" "B.Cu") (net 1))
-  (via (at 141.5 57.42) (size 0.7) (drill 0.3) (layers "F.Cu" "B.Cu") (net 1))
+  (via (at 141.489906 57.42) (size 0.7) (drill 0.3) (layers "F.Cu" "B.Cu") (net 1))
   (via (at 139.739947 67.32998) (size 0.7) (drill 0.3) (layers "F.Cu" "B.Cu") (net 1))
   (via (at 135.43 44.85) (size 0.7) (drill 0.3) (layers "F.Cu" "B.Cu") (net 1))
-  (via (at 143.67 55.2) (size 0.7) (drill 0.3) (layers "F.Cu" "B.Cu") (net 1))
+  (via (at 143.71 56.335) (size 0.7) (drill 0.3) (layers "F.Cu" "B.Cu") (net 1))
+  (via (at 142.66 57.42) (size 0.7) (drill 0.3) (layers "F.Cu" "B.Cu") (net 1))
+  (via (at 143.71 55.25) (size 0.7) (drill 0.3) (layers "F.Cu" "B.Cu") (net 1))
   (via (at 140.050013 61.507474) (size 0.7) (drill 0.3) (layers "F.Cu" "B.Cu") (net 1))
   (via (at 149.51 46.52375) (size 0.7) (drill 0.3) (layers "F.Cu" "B.Cu") (net 1))
   (via (at 149.51 50.4575) (size 0.7) (drill 0.3) (layers "F.Cu" "B.Cu") (net 1))
-  (via (at 143.69 57.45) (size 0.7) (drill 0.3) (layers "F.Cu" "B.Cu") (net 1))
+  (via (at 143.71 57.42) (size 0.7) (drill 0.3) (layers "F.Cu" "B.Cu") (net 1))
   (via (at 142.331784 50.55229) (size 0.7) (drill 0.3) (layers "F.Cu" "B.Cu") (net 1))
   (via (at 145.16 49.02) (size 0.7) (drill 0.3) (layers "F.Cu" "B.Cu") (net 1))
-  (via (at 141.489906 55.294767) (size 0.7) (drill 0.3) (layers "F.Cu" "B.Cu") (net 1))
+  (via (at 141.489906 56.335) (size 0.7) (drill 0.3) (layers "F.Cu" "B.Cu") (net 1))
+  (via (at 141.489906 55.25) (size 0.7) (drill 0.3) (layers "F.Cu" "B.Cu") (net 1))
   (via (at 149.51 51.76875) (size 0.7) (drill 0.3) (layers "F.Cu" "B.Cu") (net 1))
   (via (at 149.51 47.835) (size 0.7) (drill 0.3) (layers "F.Cu" "B.Cu") (net 1))
   (via (at 147.439998 54.305001) (size 0.7) (drill 0.3) (layers "F.Cu" "B.Cu") (net 1))
+  (via (at 142.64 55.25) (size 0.7) (drill 0.3) (layers "F.Cu" "B.Cu") (net 1))
   (via (at 149.51 49.14625) (size 0.7) (drill 0.3) (layers "F.Cu" "B.Cu") (net 1))
   (via (at 142.889968 45.4725) (size 0.7) (drill 0.3) (layers "F.Cu" "B.Cu") (net 1))
   (via (at 141.921403 43.930861) (size 0.7) (drill 0.3) (layers "F.Cu" "B.Cu") (net 1))
-  (via (at 142.680167 56.3) (size 0.7) (drill 0.3) (layers "F.Cu" "B.Cu") (net 1))
+  (via (at 142.680167 56.335) (size 0.7) (drill 0.3) (layers "F.Cu" "B.Cu") (net 1))
   (via (at 139.04 48.62) (size 0.7) (drill 0.3) (layers "F.Cu" "B.Cu") (net 1))
   (segment (start 144.4 62.3) (end 144.14 62.56) (width 0.25) (layer "B.Cu") (net 1))
