File: KiCADWork/BLEEarrings nRF52832/BLEEarrings.kicad_pcb (KiCad board)
At the start: 2 copper layers, 25.8 x 38.8 mm, 55 parts, among them J1 Screw_Terminal_01x01, J2 Screw_Terminal_01x02, J3 USB_C_Receptacle, SW1 TK-6580B-1, SW2 SW_DIP_x01, U1 MCP73831T-2ACI/OT, U2 XB6096I2SV, U3 NRF52833-QDAA-R7, Y1 XL7EL89CKI-111YLC-32M, Y2 X161032768KLD2SI

Commit message: Started mirror earrings and case
Routing:
- net +BATT: track 23.8 -> 20.9 mm
Other:
- board text removed: "Bat+"
