File: KiCADWork/Earring/Earring/Earring.kicad_sch (KiCad schematic)
At the start: 3 parts, among them J1 Screw_Terminal_01x02, J2 Screw_Terminal_01x01

Commit message: Started mirror earrings and case
Parts:
- removed J1: Screw_Terminal_01x02, easyeda2kicad:CONN-SMD_2059-302, symbol Connector:Screw_Terminal_01x02
- removed J2: Screw_Terminal_01x01, easyeda2kicad:CONN-SMD_custom1, symbol Connector:Screw_Terminal_01x01
- added TP1, TP2, TP3: TestPoint, TestPoint:TestPoint_THTPad_D1.0mm_Drill0.5mm, symbol Connector:TestPoint
Connections:
- net at D1.4 (DIN): now also TP1.1
- net at D1.1 (VDD): now also TP2.1
- net at D1.2 (DOUT), D1.3 (VSS): now also TP3.1
Changed lines of the file:
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@@
 (kicad_sch (version 20230121) (generator eeschema)
   (paper "A4")
-  (junction (at 176.53 81.28) (diameter 0) (color 0 0 0 0)
+  (junction (at 176.53 86.36) (diameter 0) (color 0 0 0 0)
   )
   (wire (pts (xy 176.53 76.2) (xy 177.165 76.2))
@@
     (stroke (width 0) (type default))
   )
-  (wire (pts (xy 176.53 78.74) (xy 176.53 81.28))
-    (stroke (width 0) (type default))
-  )
-  (wire (pts (xy 177.165 78.74) (xy 176.53 78.74))
+  (wire (pts (xy 177.8 86.36) (xy 176.53 86.36))
     (stroke (width 0) (type default))
   )
@@
     (stroke (width 0) (type default))
   )
-  (symbol (lib_id "Connector:Screw_Terminal_01x01") (at 137.16 81.28 180) (unit 1)
+  (symbol (lib_id "Connector:TestPoint") (at 142.24 81.28 90) (unit 1)
     (in_bom yes) (on_board yes) (dnp no) (fields_autoplaced)
-    (property "Reference" "J2" (at 137.16 75.565 0)
+    (property "Reference" "TP1" (at 138.938 76.2 90)
       (effects (font (size 1.27 1.27)))
     )
-    (property "Value" "Screw_Terminal_01x01" (at 137.16 78.105 0)
+    (property "Value" "TestPoint" (at 138.938 78.74 90)
       (effects (font (size 1.27 1.27)))
     )
-    (property "Footprint" "easyeda2kicad:CONN-SMD_custom1" (at 137.16 81.28 0)
+    (property "Footprint" "TestPoint:TestPoint_THTPad_D1.0mm_Drill0.5mm" (at 142.24 76.2 0)
       (effects (font (size 1.27 1.27)) hide)
     )
-    (property "Datasheet" "~" (at 137.16 81.28 0)
+    (property "Datasheet" "~" (at 142.24 76.2 0)
       (effects (font (size 1.27 1.27)) hide)
     )
@@
       (project "Earring"
         (path "/7ade6d1b-326a-48c0-91fe-d3024994d83d"
-          (reference "J2") (unit 1)
+          (reference "TP1") (unit 1)
+        )
+      )
+    )
+  )
+  (symbol (lib_id "Connector:TestPoint") (at 177.165 76.2 270) (unit 1)
+    (in_bom yes) (on_board yes) (dnp no) (fields_autoplaced)
+    (property "Reference" "TP2" (at 182.245 74.93 90)
+      (effects (font (size 1.27 1.27)) (justify left))
+    )
+    (property "Value" "TestPoint" (at 182.245 77.47 90)
+      (effects (font (size 1.27 1.27)) (justify left))
+    )
+    (property "Footprint" "TestPoint:TestPoint_THTPad_D1.0mm_Drill0.5mm" (at 177.165 81.28 0)
+      (effects (font (size 1.27 1.27)) hide)
+    )
+    (property "Datasheet" "~" (at 177.165 81.28 0)
+      (effects (font (size 1.27 1.27)) hide)
+    )
+    (pin "1")
+    (instances
+      (project "Earring"
+        (path "/7ade6d1b-326a-48c0-91fe-d3024994d83d"
+          (reference "TP2") (unit 1)
         )
       )
@@
     )
   )
-  (symbol (lib_id "Connector:Screw_Terminal_01x02") (at 182.245 76.2 0) (unit 1)
+  (symbol (lib_id "Connector:TestPoint") (at 177.8 86.36 270) (unit 1)
     (in_bom yes) (on_board yes) (dnp no) (fields_autoplaced)
-    (property "Reference" "J1" (at 184.785 76.2 0)
+    (property "Reference" "TP3" (at 183.515 85.09 90)
       (effects (font (size 1.27 1.27)) (justify left))
     )
-    (property "Value" "Screw_Terminal_01x02" (at 184.785 78.74 0)
+    (property "Value" "TestPoint" (at 183.515 87.63 90)
       (effects (font (size 1.27 1.27)) (justify left))
     )
-    (property "Footprint" "easyeda2kicad:CONN-SMD_2059-302" (at 182.245 76.2 0)
+    (property "Footprint" "TestPoint:TestPoint_THTPad_D1.0mm_Drill0.5mm" (at 177.8 91.44 0)
       (effects (font (size 1.27 1.27)) hide)
     )
-    (property "Datasheet" "~" (at 182.245 76.2 0)
+    (property "Datasheet" "~" (at 177.8 91.44 0)
       (effects (font (size 1.27 1.27)) hide)
     )
     (pin "1")
-    (pin "2")
     (instances
       (project "Earring"
         (path "/7ade6d1b-326a-48c0-91fe-d3024994d83d"
-          (reference "J1") (unit 1)
+          (reference "TP3") (unit 1)
         )
       )
